Commit message: ros2-brfirst time

File: urdf/dogai.urdf (robot description, URDF)
Before this commit: robot dogai, 13 links, 12 joints
Links:
- added link world
Joints:
- added joint dummy_joint: type floating, parent world, child body, origin xyz=0 0 0.05 rpy=0 0 0

Commit message: leg_bl

File: urdf/dogai.urdf (robot description, URDF)
Before this commit: robot dogai, 14 links, 13 joints
Links:
- link leg_fr: mass 0.194 -> 0.193999611092193
- link shoulder_fr: mass 0.10629 -> 0.106289004701676
Joints:
- joint foreleg_bl_j: origin xyz=-0.0291684099209072 -0.104 -0.015 rpy=-1.5707963267949 0.143242948811687 -1.5707963267949 -> xyz=0.104 0.015 0 rpy=0 0 0.14324
- joint foreleg_fl_j: origin xyz=0.105076162853427 0 0 rpy=0 0 0 -> xyz=0.10508 0 0 rpy=0 0 0
- joint foreleg_fr_j: origin xyz=0.105076162853427 0 0 rpy=0 0 0 -> xyz=0.10508 0 0 rpy=0 0 0
- joint leg_bl_j: axis -1 0 0 -> 0 0 -1; origin xyz=0.0115 0.0293315900790929 0 rpy=2.99834970477811 0 -1.5707963267949 -> xyz=0.0115 0.0585 0 rpy=1.5708 0.14324 0
- joint leg_br_j: origin xyz=0.0115 -0.0585 0 rpy=1.5707963267949 0 0 -> xyz=0.0115 -0.0585 0 rpy=1.5708 0 0
- joint leg_fl_j: origin xyz=0.0115 0.0585000000000001 0 rpy=1.5707963267949 0 0 -> xyz=0.0115 0.0585 0 rpy=1.5708 0 0
- joint leg_fr_j: origin xyz=0.0115 -0.0584999999999999 0 rpy=1.5707963267949 0 0 -> xyz=0.0115 -0.0585 0 rpy=1.5708 0 0
- joint shoulder_fl_j: origin xyz=-0.0275 0.039 0.00800000000000001 rpy=0 1.5707963267949 0 -> xyz=-0.0275 0.039 0.008 rpy=0 1.5708 0
- joint shoulder_fr_j: origin xyz=-0.0275 -0.039 0.00800000000000003 rpy=0 1.5707963267949 0 -> xyz=-0.0275 -0.039 0.008 rpy=0 1.5708 0

Commit message: editing rviz config

File: urdf/dogai.urdf (robot description, URDF)
Before this commit: robot dogai, 13 links, 12 joints
Links:
- added link dummy_link; visual box size=0.05 0.05 0.01
Joints:
- added joint dummy_joint: type fixed, parent dummy_link, child body, origin xyz=0 0 0.25 rpy=0 0 0

Commit message: editing rviz config (ros2)

File: urdf/dogai.urdf (robot description, URDF)
Before this commit: robot dogai, 14 links, 13 joints
Links:
- removed link world
- added link dummy_link; visual box size=0.05 0.05 0.01
Joints:
- joint dummy_joint: origin xyz=0 0 0.05 rpy=0 0 0 -> xyz=0 0 0.25 rpy=0 0 0; parent world -> dummy_link; type floating -> fixed

Commit message: ---

File: urdf/dogai.urdf (robot description, URDF)
Before this commit: robot dogai, 14 links, 13 joints
Links:
- removed link dummy_link
- added link world
Joints:
- joint dummy_joint: parent dummy_link -> world

Commit message: ===

File: urdf/dogai.urdf (robot description, URDF)
Before this commit: robot dogai, 13 links, 12 joints
Links:
- added link world
Joints:
- added joint dummy_joint: type fixed, parent world, child body, origin xyz=0 0 0.25 rpy=0 0 0
